File: pcb/fusioncore.sch (KiCad schematic (older format))
At the start: 104 parts, among them J1 Conn_02x12_Top_Bottom, J10 Pump_Misc_1, J11 Pump_Misc_2, J12 Flow_Warm, J13 Flow_Cold, J14 Trigger, J15 Valve_M1, J16 Valve_M2, J17 Valve_M3, J18 Valve_M4, J19 Valve_Air_Lime, J2 Temp_1, J20 Valve_Air_Rum, J21 Valve_Air_Out, J22 LED, J3 40HAT, J4 Temp_2, J5 WEIGHT, J6 Pump_Water_Cold, J7 Pump_Water_Warm, J8 Pump_Air, J9 CONN_01X02, Q1 DMG2305UX, Q10 AO3400A, Q11 AO3400A, Q12 AO3400A, Q13 AO3400A, Q14 AO3400A, Q16 MMBT4403, Q2 DMMT5401, Q3 AO3400A, Q4 AO3400A, Q5 AO3400A, Q6 AO3400A, Q7 AO3400A, Q8 AO3400A, Q9 AO3400A, SW1 POWER_ON, U1 HX711, U2 CAT24C32, U3 LTC2990, U4 LTC2990

Commit message: Organize the schema
Other:
- note added: "Current Sensor"
- note added: "Voltage Sensor"
- note removed: "Current/Voltage Sensor"
- note removed: "EEPROM WRITE ENABLE"
- moved on the sheet: C6, C7, J12, J13, Q1, Q2A, Q2B, R16, R17, R18, R19, R2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

Commit message: Working on replacing some 2-Port Valves
Parts:
- removed D1, D2, D3, D4: D, Diode_SMD:D_SOD-123F, symbol Device:D_Small
- removed J15: Valve_M1, TerminalBlock_Phoenix:TerminalBlock_Phoenix_PT-1,5-2-5.0-H_1x02_P5.00mm_Horizontal, symbol Connector:Screw_Terminal_01x02
- removed J16: Valve_M2, TerminalBlock_Phoenix:TerminalBlock_Phoenix_PT-1,5-2-5.0-H_1x02_P5.00mm_Horizontal, symbol Connector:Screw_Terminal_01x02
- removed J17: Valve_M3, TerminalBlock_Phoenix:TerminalBlock_Phoenix_PT-1,5-2-5.0-H_1x02_P5.00mm_Horizontal, symbol Connector:Screw_Terminal_01x02
- removed J18: Valve_M4, TerminalBlock_Phoenix:TerminalBlock_Phoenix_PT-1,5-2-5.0-H_1x02_P5.00mm_Horizontal, symbol Connector:Screw_Terminal_01x02
- removed J4: Temp_2, TerminalBlock_Phoenix:TerminalBlock_Phoenix_PT-1,5-3-5.0-H_1x03_P5.00mm_Horizontal, symbol Connector:Screw_Terminal_01x03
- removed Q10, Q11, Q8, Q9: AO3400A, Package_TO_SOT_SMD:SOT-23, symbol misc:AO3400A
- added D? (x8): LED, Resistor_SMD:R_0603_1608Metric_Pad1.05x0.95mm_HandSolder, symbol Device:LED
- added J?: Valve_M4, TerminalBlock_Phoenix:TerminalBlock_Phoenix_PT-1,5-3-5.0-H_1x03_P5.00mm_Horizontal, symbol Connector:Screw_Terminal_01x03
- added J?: Valve_M3, TerminalBlock_Phoenix:TerminalBlock_Phoenix_PT-1,5-3-5.0-H_1x03_P5.00mm_Horizontal, symbol Connector:Screw_Terminal_01x03
- added J?: Valve_M2, TerminalBlock_Phoenix:TerminalBlock_Phoenix_PT-1,5-3-5.0-H_1x03_P5.00mm_Horizontal, symbol Connector:Screw_Terminal_01x03
- added J?: Valve_M1, TerminalBlock_Phoenix:TerminalBlock_Phoenix_PT-1,5-3-5.0-H_1x03_P5.00mm_Horizontal, symbol Connector:Screw_Terminal_01x03
- added R? (x8): 360, Resistor_SMD:R_0603_1608Metric_Pad1.05x0.95mm_HandSolder, symbol Device:R
- U5: renamed from U?; LCSC (none) -> C53406
Connections:
- net 12V: now also R?.2, R?.2, R?.2, R?.2, R?.2, R?.2, R?.2, R?.2
- net 5V: now also J?.3 (Pin_3), J?.3 (Pin_3), J?.3 (Pin_3), J?.3 (Pin_3)
- net GND: now also J?.1 (Pin_1), J?.1 (Pin_1), J?.1 (Pin_1), J?.1 (Pin_1)
- net Valve_M1: now also U5.4 (A4)
- net Valve_M2: now also U5.7 (A5)
- net Valve_M3: now also U5.8 (A6)
- net Valve_M4: now also U5.9 (A7)
- net at D8.2 (A), J6.2 (Pin_2), Q3.3 (D): now also D?.1 (K)
- net at D9.2 (A), J7.2 (Pin_2), Q4.3 (D): now also D?.1 (K)
- net at D10.2 (A), J8.2 (Pin_2), Q5.3 (D): now also D?.1 (K)
- net at D11.2 (A), J10.2 (Pin_2), Q6.3 (D): now also D?.1 (K)
- net at D12.2 (A), J11.2 (Pin_2), Q7.3 (D): now also D?.1 (K)
- net Valve_M4_5V: now reaches U5.12 (B7)
- net Valve_M4_5V: now also J?.2 (Pin_2)
- net Valve_M3_5V: now reaches U5.13 (B6)
- net Valve_M3_5V: now also J?.2 (Pin_2)
- net Valve_M2_5V: now reaches U5.14 (B5)
- net Valve_M2_5V: now also J?.2 (Pin_2)
- net Valve_M1_5V: now reaches U5.17 (B4)
- net Valve_M1_5V: now also J?.2 (Pin_2)
- net at D7.2 (A), J21.2 (Pin_2), Q14.3 (D): now also D?.1 (K)
- net at D6.2 (A), J20.2 (Pin_2), Q13.3 (D): now also D?.1 (K)
- net at D5.2 (A), J19.2 (Pin_2), Q12.3 (D): now also D?.1 (K)
- new net: D?.2 (A), R?.1 (x8)
- no-connect marks 9 -> 11
Other:
- note added: "Valve Servos"
- moved on the sheet: D5, D6, D7, J19, J20, J21, Q12, Q13, Q14

Commit message: Finalized current PCB iteration
Parts:
- removed R33: DNP, Resistor_SMD:R_0805_2012Metric_Pad1.15x1.40mm_HandSolder, symbol Device:R
- added JP1, JP2: SolderJumper_2_Open, Jumper:SolderJumper-2_P1.3mm_Open_Pad1.0x1.5mm, symbol Jumper:SolderJumper_2_Open
- D13: value POWER GOOD -> PWG
- D14: value STANDBY -> STB
- J2: value Temp_1 -> Temperature
- J6: value Pump_Water_Cold -> Pump_Cold
- J7: value Pump_Water_Warm -> Pump_Warm
- R11: value DNP -> 10K; LCSC (none) -> C17414
- R16: footprint Resistor_SMD:R_2512_6332Metric_Pad1.52x3.35mm_HandSolder -> Resistor_SMD:R_1206_3216Metric_Pad1.42x1.75mm_HandSolder
- TP1, TP2, TP3, TP4, TP5: footprint TestPoint:TestPoint_Plated_Hole_D2.0mm -> TestPoint:TestPoint_THTPad_D2.0mm_Drill1.0mm
- gave numbers to parts that had none: 20
Connections:
- net 3V3: now also R11.2, U5.6 (OE)
- net 5V: now also JP2.1 (A)
- net 5V_PI: now also JP2.2 (B)
- net Flow_C: now also U5.9 (A7); no longer U5.3 (A3)
- net Flow_C_5V: now also U5.12 (B7); no longer U5.18 (B3)
- net Flow_W: now also U5.8 (A6); no longer U5.2 (A2)
- net Flow_W_5V: now also U5.13 (B6); no longer U5.19 (B2)
- net GND: now also R11.1, JP1.1 (A); no longer R11.2
- net LED_PWM: now also U5.10 (A8); no longer U5.1 (A1)
- net LED_PWM_5V: now also U5.11 (B8); no longer U5.20 (B1)
- net Valve_M1: now also U5.1 (A1); no longer U5.4 (A4)
- net Valve_M1_5V: now also U5.20 (B1); no longer U5.17 (B4)
- net Valve_M2: now also U5.2 (A2); no longer U5.7 (A5)
- net Valve_M2_5V: now also U5.19 (B2); no longer U5.14 (B5)
- net Valve_M3: now also U5.3 (A3); no longer U5.8 (A6)
- net Valve_M3_5V: now also U5.18 (B3); no longer U5.13 (B6)
- net Valve_M4: now also U5.4 (A4); no longer U5.9 (A7)
- net Valve_M4_5V: now also U5.17 (B4); no longer U5.12 (B7)
- net at J9.2 (Pin_2), R29.2, U2.7 (WP): now also JP1.2 (B); no longer R11.1

Commit message: Fixed some more issues on pcb
Parts:
- D1, D15, D16, D17, D18, D2, D3, D4: footprint Resistor_SMD:R_0603_1608Metric_Pad1.05x0.95mm_HandSolder -> LED_SMD:LED_0603_1608Metric_Pad1.05x0.95mm_HandSolder
- U5: footprint Package_SON:USON-20_2x4mm_P0.4mm -> Package_SO:TSSOP-20_4.4x6.5mm_P0.65mm
Changed lines of the file:
@@
 F 0 "U5" H 1400 6161 50  0000 C CNN
 F 1 "TXB0108DQSR" H 1400 6070 50  0000 C CNN
-F 2 "Package_SON:USON-20_2x4mm_P0.4mm" H 1400 6200 50  0001 C CNN
+F 2 "Package_SO:TSSOP-20_4.4x6.5mm_P0.65mm" H 1400 6200 50  0001 C CNN
 F 3 "http://www.ti.com/lit/ds/symlink/txb0108.pdf" H 1400 6850 50  0001 C CNN
 F 4 "C53406" H 1400 6950 50  0001 C CNN "LCSC"
@@
 F 0 "D3" H 11000 9900 50  0000 C CNN
 F 1 "LED" H 11150 10050 50  0001 C CNN
-F 2 "Resistor_SMD:R_0603_1608Metric_Pad1.05x0.95mm_HandSolder" H 11000 10000 50  0001 C CNN
+F 2 "LED_SMD:LED_0603_1608Metric_Pad1.05x0.95mm_HandSolder" H 11000 10000 50  0001 C CNN
 F 3 "https://datasheet.lcsc.com/szlcsc/Everlight-Elec-19-217-BHC-ZL1M2RY-3T_C72041.pdf" H 11000 10000 50  0001 C CNN
 F 4 "C72041" H 11000 10000 50  0001 C CNN "LCSC"
@@
 F 0 "D2" V 10650 9750 50  0000 C CNN
 F 1 "LED" V 10650 9750 50  0001 C CNN
-F 2 "Resistor_SMD:R_0603_1608Metric_Pad1.05x0.95mm_HandSolder" H 10650 9850 50  0001 C CNN
+F 2 "LED_SMD:LED_0603_1608Metric_Pad1.05x0.95mm_HandSolder" H 10650 9850 50  0001 C CNN
 F 3 "https://datasheet.lcsc.com/szlcsc/Everlight-Elec-19-217-BHC-ZL1M2RY-3T_C72041.pdf" H 10650 9850 50  0001 C CNN
 F 4 "C72041" H 10650 9850 50  0001 C CNN "LCSC"
@@
 F 0 "D1" V 10300 9750 50  0000 C CNN
 F 1 "LED" V 10300 9750 50  0001 C CNN
-F 2 "Resistor_SMD:R_0603_1608Metric_Pad1.05x0.95mm_HandSolder" H 10300 9850 50  0001 C CNN
+F 2 "LED_SMD:LED_0603_1608Metric_Pad1.05x0.95mm_HandSolder" H 10300 9850 50  0001 C CNN
 F 3 "https://datasheet.lcsc.com/szlcsc/Everlight-Elec-19-217-BHC-ZL1M2RY-3T_C72041.pdf" H 10300 9850 50  0001 C CNN
 F 4 "C72041" H 10300 9850 50  0001 C CNN "LCSC"
@@
 F 0 "D4" H 12750 5400 50  0000 C CNN
 F 1 "LED" H 13000 5400 50  0001 C CNN
-F 2 "Resistor_SMD:R_0603_1608Metric_Pad1.05x0.95mm_HandSolder" H 12850 5350 50  0001 C CNN
+F 2 "LED_SMD:LED_0603_1608Metric_Pad1.05x0.95mm_HandSolder" H 12850 5350 50  0001 C CNN
 F 3 "https://datasheet.lcsc.com/szlcsc/Everlight-Elec-19-217-BHC-ZL1M2RY-3T_C72041.pdf" H 12850 5350 50  0001 C CNN
 F 4 "C72041" H 12850 5350 50  0001 C CNN "LCSC"
@@
 F 0 "D15" H 12750 5700 50  0000 C CNN
 F 1 "LED" H 13000 5700 50  0001 C CNN
-F 2 "Resistor_SMD:R_0603_1608Metric_Pad1.05x0.95mm_HandSolder" H 12850 5650 50  0001 C CNN
+F 2 "LED_SMD:LED_0603_1608Metric_Pad1.05x0.95mm_HandSolder" H 12850 5650 50  0001 C CNN
 F 3 "https://datasheet.lcsc.com/szlcsc/Everlight-Elec-19-217-BHC-ZL1M2RY-3T_C72041.pdf" H 12850 5650 50  0001 C CNN
 F 4 "C72041" H 12850 5650 50  0001 C CNN "LCSC"
@@
 F 0 "D16" H 12750 6000 50  0000 C CNN
 F 1 "LED" H 13000 6000 50  0001 C CNN
-F 2 "Resistor_SMD:R_0603_1608Metric_Pad1.05x0.95mm_HandSolder" H 12850 5950 50  0001 C CNN
+F 2 "LED_SMD:LED_0603_1608Metric_Pad1.05x0.95mm_HandSolder" H 12850 5950 50  0001 C CNN
 F 3 "https://datasheet.lcsc.com/szlcsc/Everlight-Elec-19-217-BHC-ZL1M2RY-3T_C72041.pdf" H 12850 5950 50  0001 C CNN
 F 4 "C72041" H 12850 5950 50  0001 C CNN "LCSC"
@@
 F 0 "D17" H 12750 6300 50  0000 C CNN
 F 1 "LED" H 13000 6300 50  0001 C CNN
-F 2 "Resistor_SMD:R_0603_1608Metric_Pad1.05x0.95mm_HandSolder" H 12850 6250 50  0001 C CNN
+F 2 "LED_SMD:LED_0603_1608Metric_Pad1.05x0.95mm_HandSolder" H 12850 6250 50  0001 C CNN
 F 3 "https://datasheet.lcsc.com/szlcsc/Everlight-Elec-19-217-BHC-ZL1M2RY-3T_C72041.pdf" H 12850 6250 50  0001 C CNN
 F 4 "C72041" H 12850 6250 50  0001 C CNN "LCSC"
@@
 F 0 "D18" H 12750 6600 50  0000 C CNN
 F 1 "LED" H 13000 6600 50  0001 C CNN
-F 2 "Resistor_SMD:R_0603_1608Metric_Pad1.05x0.95mm_HandSolder" H 12850 6550 50  0001 C CNN
+F 2 "LED_SMD:LED_0603_1608Metric_Pad1.05x0.95mm_HandSolder" H 12850 6550 50  0001 C CNN
 F 3 "https://datasheet.lcsc.com/szlcsc/Everlight-Elec-19-217-BHC-ZL1M2RY-3T_C72041.pdf" H 12850 6550 50  0001 C CNN
 F 4 "C72041" H 12850 6550 50  0001 C CNN "LCSC"

Commit message: Added more debug and expansion connectors
Parts:
- added J18: Conn_02x03_Top_Bottom, Connector_Molex:Molex_Micro-Fit_3.0_43045-0612_2x03_P3.00mm_Vertical, symbol Connector_Generic:Conn_02x03_Top_Bottom
- added J23: I2C_DBG, Connector_PinHeader_2.54mm:PinHeader_1x02_P2.54mm_Vertical, symbol Connector_Generic:Conn_01x02
- SW1: footprint (none) -> Button_Switch_THT:SW_CuK_JS202011CQN_DPDT_Straight; symbol Switch:SW_DIP_x01 -> Switch:SW_SPDT; Digikey (none) -> 401-2001-ND
- U2: LCSC (none) -> C81193
Connections:
- net 12V: now also J18.4 (Pin_4)
- net 5V: now also J18.6 (Pin_6)
- net GND: now also SW1.3 (C), J18.2 (Pin_2), J18.5 (Pin_5); no longer SW1.2
- net I2C_SCL: now also J18.1 (Pin_1), J23.1 (Pin_1)
- net I2C_SDA: now also J18.3 (Pin_3), J23.2 (Pin_2)
- net PS_ON: now also SW1.2 (B); no longer SW1.1
Other:
- note added: "Expansion Connector"
- moved on the sheet: TP1, TP2, TP3, TP4, TP5
Changed lines of the file:
@@
 F 1 "CAT24C32" H 1750 4950 50  0000 C CNN
 F 2 "Package_SOIC:SOIC-8_3.9x4.9mm_P1.27mm" H 2000 4600 50  0001 C CNN
-F 3 "" H 2000 4600 50  0000 C CNN
+F 3 "https://datasheet.lcsc.com/szlcsc/1809291220_ON-Semicon-CAT24C32WI-GT3_C81193.pdf" H 2000 4600 50  0001 C CNN
+F 4 "C81193" H 2000 4600 50  0001 C CNN "LCSC"
 	1    2000 4600
 	1    0    0    -1
@@
 	12550 2150 13300 2150
 $Comp
-L Switch:SW_DIP_x01 SW1
+L Switch:SW_SPDT SW1
 U 1 1 5F9F56A0
-P 15350 1650
-F 0 "SW1" H 15350 1917 50  0000 C CNN
-F 1 "POWER_ON" H 15350 1826 50  0000 C CNN
-F 2 "" H 15350 1650 50  0001 C CNN
-F 3 "~" H 15350 1650 50  0001 C CNN
-	1    15350 1650
+P 15250 1650
+F 0 "SW1" H 15250 1917 50  0000 C CNN
+F 1 "POWER_ON" H 15250 1826 50  0000 C CNN
+F 2 "Button_Switch_THT:SW_CuK_JS202011CQN_DPDT_Straight" H 15250 1650 50  0001 C CNN
+F 3 "https://dznh3ojzb2azq.cloudfront.net/products/Slide/JS/documents/datasheet.pdf" H 15250 1650 50  0001 C CNN
+F 4 "401-2001-ND" H 15250 1650 50  0001 C CNN "Digikey"
+	1    15250 1650
 	1    0    0    -1
 $EndComp
@@
 L power:GND #PWR0104
 U 1 1 5F9F724F
-P 15850 1650
-F 0 "#PWR0104" H 15850 1400 50  0001 C CNN
-F 1 "GND" H 15855 1477 50  0000 C CNN
-F 2 "" H 15850 1650 50  0001 C CNN
-F 3 "" H 15850 1650 50  0001 C CNN
-	1    15850 1650
+P 15650 1750
+F 0 "#PWR0104" H 15650 1500 50  0001 C CNN
+F 1 "GND" H 15655 1577 50  0000 C CNN
+F 2 "" H 15650 1750 50  0001 C CNN
+F 3 "" H 15650 1750 50  0001 C CNN
+	1    15650 1750
 	1    0    0    -1
 $EndComp
@@
 	13800 1650 15050 1650
 Wire Wire Line
-	15650 1650 15850 1650
+	15450 1750 15650 1750
 Connection ~ 11950 3650
 Connection ~ 11950 4100
@@
 L Connector:TestPoint TP2
 U 1 1 5E238E97
+P 3650 6050
+F 0 "TP2" V 3604 6238 50  0000 L CNN
+F 1 "3V3_PI" V 3695 6238 50  0000 L CNN
+F 2 "TestPoint:TestPoint_THTPad_D2.0mm_Drill1.0mm" H 3850 6050 50  0001 C CNN
+F 3 "~" H 3850 6050 50  0001 C CNN
+	1    3650 6050
+	0    1    1    0
+$EndComp
+$Comp
+L Connector:TestPoint TP3
+U 1 1 5E238B2E
+P 3650 6250
+F 0 "TP3" V 3604 6438 50  0000 L CNN
+F 1 "3V3" V 3695 6438 50  0000 L CNN
+F 2 "TestPoint:TestPoint_THTPad_D2.0mm_Drill1.0mm" H 3850 6250 50  0001 C CNN
+F 3 "~" H 3850 6250 50  0001 C CNN
+	1    3650 6250
+	0    1    1    0
+$EndComp
+$Comp
+L Connector:TestPoint TP4
+U 1 1 5E2387C0
+P 3650 6450
+F 0 "TP4" V 3604 6638 50  0000 L CNN
+F 1 "5V" V 3695 6638 50  0000 L CNN
+F 2 "TestPoint:TestPoint_THTPad_D2.0mm_Drill1.0mm" H 3850 6450 50  0001 C CNN
+F 3 "~" H 3850 6450 50  0001 C CNN
+	1    3650 6450
+	0    1    1    0
+$EndComp
+$Comp
+L Connector:TestPoint TP5
+U 1 1 5E236258
 P 3650 6650
-F 0 "TP2" V 3604 6838 50  0000 L CNN
-F 1 "3V3_PI" V 3695 6838 50  0000 L CNN
+F 0 "TP5" V 3604 6838 50  0000 L CNN
+F 1 "12V" V 3695 6838 50  0000 L CNN
 F 2 "TestPoint:TestPoint_THTPad_D2.0mm_Drill1.0mm" H 3850 6650 50  0001 C CNN
 F 3 "~" H 3850 6650 50  0001 C CNN
@@
 $EndComp
 $Comp
-L Connector:TestPoint TP3
-U 1 1 5E238B2E
-P 3650 6850
-F 0 "TP3" V 3604 7038 50  0000 L CNN
-F 1 "3V3" V 3695 7038 50  0000 L CNN
-F 2 "TestPoint:TestPoint_THTPad_D2.0mm_Drill1.0mm" H 3850 6850 50  0001 C CNN
-F 3 "~" H 3850 6850 50  0001 C CNN
-	1    3650 6850
-	0    1    1    0
-$EndComp
-$Comp
-L Connector:TestPoint TP4
-U 1 1 5E2387C0
-P 3650 7050
-F 0 "TP4" V 3604 7238 50  0000 L CNN
-F 1 "5V" V 3695 7238 50  0000 L CNN
-F 2 "TestPoint:TestPoint_THTPad_D2.0mm_Drill1.0mm" H 3850 7050 50  0001 C CNN
-F 3 "~" H 3850 7050 50  0001 C CNN
-	1    3650 7050
-	0    1    1    0
-$EndComp
-$Comp
-L Connector:TestPoint TP5
-U 1 1 5E236258
-P 3650 7250
-F 0 "TP5" V 3604 7438 50  0000 L CNN
-F 1 "12V" V 3695 7438 50  0000 L CNN
-F 2 "TestPoint:TestPoint_THTPad_D2.0mm_Drill1.0mm" H 3850 7250 50  0001 C CNN
-F 3 "~" H 3850 7250 50  0001 C CNN
-	1    3650 7250
-	0    1    1    0
-$EndComp
-$Comp
 L Connector:TestPoint TP1
 U 1 1 5E427CC4
-P 3650 6450
-F 0 "TP1" V 3604 6638 50  0000 L CNN
-F 1 "GND" V 3695 6638 50  0000 L CNN
-F 2 "TestPoint:TestPoint_THTPad_D2.0mm_Drill1.0mm" H 3850 6450 50  0001 C CNN
-F 3 "~" H 3850 6450 50  0001 C CNN
-	1    3650 6450
-	0    1    1    0
-$EndComp
+P 3650 5850
+F 0 "TP1" V 3604 6038 50  0000 L CNN
+F 1 "GND" V 3695 6038 50  0000 L CNN
+F 2 "TestPoint:TestPoint_THTPad_D2.0mm_Drill1.0mm" H 3850 5850 50  0001 C CNN
+F 3 "~" H 3850 5850 50  0001 C CNN
+	1    3650 5850
+	0    1    1    0
+$EndComp
+Wire Wire Line
+	3650 5850 3050 5850
+Wire Wire Line
+	3650 6050 3050 6050
+Wire Wire Line
+	3650 6250 3050 6250
 Wire Wire Line
 	3650 6450 3050 6450
 Wire Wire Line
 	3650 6650 3050 6650
-Wire Wire Line
-	3650 6850 3050 6850
-Wire Wire Line
-	3650 7050 3050 7050
-Wire Wire Line
-	3650 7250 3050 7250
 $Comp
 L power:GND #PWR0114
 U 1 1 5E560038
-P 3050 6450
-F 0 "#PWR0114" H 3050 6200 50  0001 C CNN
-F 1 "GND" V 3055 6322 50  0000 R CNN
-F 2 "" H 3050 6450 50  0001 C CNN
-F 3 "" H 3050 6450 50  0001 C CNN
-	1    3050 6450
-	0    1    1    0
-$EndComp
+P 3050 5850
+F 0 "#PWR0114" H 3050 5600 50  0001 C CNN
+F 1 "GND" V 3055 5722 50  0000 R CNN
+F 2 "" H 3050 5850 50  0001 C CNN
+F 3 "" H 3050 5850 50  0001 C CNN
+	1    3050 5850
+	0    1    1    0
+$EndComp
+Text Label 3050 6050 0    50   ~ 0
+3V3_PI
+Text Label 3050 6250 0    50   ~ 0
+3V3
+Text Label 3050 6450 0    50   ~ 0
+5V
 Text Label 3050 6650 0    50   ~ 0
-3V3_PI
-Text Label 3050 6850 0    50   ~ 0
-3V3
-Text Label 3050 7050 0    50   ~ 0
-5V
-Text Label 3050 7250 0    50   ~ 0
 12V
 Text Notes 3000 5750 0    118  ~ 24
@@
 $EndComp
 Connection ~ 1000 6250
+Wire Notes Line
+	2650 7250 4400 7250
+Text Notes 2700 7450 0    102  ~ 20
+Expansion Connector
+$Comp
+L Connector_Generic:Conn_02x03_Top_Bottom J18
+U 1 1 5E55E4B6
+P 3450 7950
+F 0 "J18" H 3500 8267 50  0000 C CNN
+F 1 "Conn_02x03_Top_Bottom" H 3500 8176 50  0000 C CNN
+F 2 "Connector_Molex:Molex_Micro-Fit_3.0_43045-0612_2x03_P3.00mm_Vertical" H 3450 7950 50  0001 C CNN
+F 3 "https://www.molex.com/pdm_docs/sd/430450612_sd.pdf" H 3450 7950 50  0001 C CNN
+F 4 "WM1791-ND " H 3450 7950 50  0001 C CNN "Digikey"
+	1    3450 7950
+	1    0    0    -1
+$EndComp
+Wire Wire Line
+	3250 7850 2700 7850
+Wire Wire Line
+	3250 7950 2700 7950
+Wire Wire Line
+	3250 8050 2700 8050
+Wire Wire Line
+	3750 8050 4350 8050
+Wire Wire Line
+	3750 7950 4350 7950
+Text Label 2700 7850 0    50   ~ 0
+I2C_SCL
+Text Label 2700 8050 0    50   ~ 0
+I2C_SDA
+Text Label 4350 8050 2    50   ~ 0
+5V
+Text Label 4350 7850 2    50   ~ 0
+12V
+Text Label 4350 7950 2    50   ~ 0
+GND
+Text Label 2700 7950 0    50   ~ 0
+GND
+Wire Wire Line
+	3750 7850 4350 7850
+$Comp
+L Connector_Generic:Conn_01x02 J23
+U 1 1 5E8D6410
+P 3850 6950
+F 0 "J23" V 3950 6900 50  0000 C CNN
+F 1 "I2C_DBG" V 4050 6900 50  0000 C CNN
+F 2 "Connector_PinHeader_2.54mm:PinHeader_1x02_P2.54mm_Vertical" H 3850 6950 50  0001 C CNN
+F 3 "" H 3850 6950 50  0000 C CNN
+	1    3850 6950
+	1    0    0    -1
+$EndComp
+Wire Wire Line
+	3650 6950 3050 6950
+Wire Wire Line
+	3650 7050 3050 7050
+Text Label 3050 6950 0    50   ~ 0
+I2C_SCL
+Text Label 3050 7050 0    50   ~ 0
+I2C_SDA
 $EndSCHEMATC
